File: ReferencniDizajn/reference-power.kicad_sch (KiCad schematic)
At the start: 9 parts, among them J1 USB_C_Receptacle_USB2.0_16P, U1 USBLC6-2SC6, U2 XC6220B331MR

Commit message: first commit
Connections:
- net USB_D+: no longer J1.A6 (D+), J1.B6 (D+), U1.3 (I/O2)
- net USB_D-: no longer J1.A7 (D-), J1.B7 (D-), U1.1 (I/O1)
- new net D+: J1.A6 (D+), J1.B6 (D+), U1.3 (I/O2)
- new net D-: J1.A7 (D-), J1.B7 (D-), U1.1 (I/O1)
Changed lines of the file:
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@@
 		(date "2026-08-28")
 		(company "UL FRI")
-		(comment 1 "Ime Priimek")
+		(comment 1 "Pa3cio")
 	)
 	(rectangle
@@
 		)
 	)
-	(global_label "USB_D-"
-		(shape input)
-		(at 80.01 58.42 90)
-		(fields_autoplaced yes)
+	(label "D+"
+		(at 83.82 60.96 0)
 		(effects
 			(font
 				(size 1.27 1.27)
 			)
-			(justify left)
-		)
-		(property "Intersheetrefs" "${INTERSHEET_REFS}"
-			(at 80.01 47.8148 90)
-			(show_name no)
-			(do_not_autoplace no)
-			(effects
-				(font
-					(size 1.27 1.27)
-				)
-				(justify left)
-			)
-		)
-	)
-	(global_label "USB_D+"
-		(shape input)
-		(at 58.42 60.96 270)
-		(fields_autoplaced yes)
+			(justify left bottom)
+		)
+	)
+	(label "D-"
+		(at 83.82 58.42 0)
 		(effects
 			(font
 				(size 1.27 1.27)
 			)
-			(justify right)
-		)
-		(property "Intersheetrefs" "${INTERSHEET_REFS}"
-			(at 58.42 71.5652 90)
-			(show_name no)
-			(do_not_autoplace no)
-			(effects
-				(font
-					(size 1.27 1.27)
-				)
-				(justify right)
-			)
-		)
-	)
+			(justify left bottom)
+		)
+	)
