File: 02-postavitev/FRI-ESP32.kicad_pcb (KiCad board)
At the start: 4 copper layers, 34.9 x 48.5 mm, 29 parts, among them J1 USB_C_Receptacle_USB2.0_16P, J2 Conn_01x08, J3 Conn_01x08, U1 USBLC6-2SC6, U2 XC6220B331MR, U3 ESP32-C3-MINI-1

Commit message: Popravljam sedkcije in dodajam slike z handbook
Parts:
- added REF**: Fiducial_1mm_Mask2mm, Fiducial:Fiducial_1mm_Mask2mm, F.Cu at (234.0, 126.7)
- added REF**: Fiducial_1mm_Mask2mm, Fiducial:Fiducial_1mm_Mask2mm, F.Cu at (202.9, 126.9)
- added REF**: Fiducial_1mm_Mask2mm, Fiducial:Fiducial_1mm_Mask2mm, F.Cu at (203.0, 87.6)
- moved RESET1 6.71 mm to (204.4, 117.6)
- moved C3 6.71 mm to (204.5, 120.4)
- moved R4 6.71 mm to (205.8, 115.4)
- moved BOOT1 6.61 mm to (231.2, 117.4)
- moved C4 6.61 mm to (231.1, 120.2)
- moved R5 6.61 mm to (232.6, 115.2)
