File: 04-rutano/FRI-ESP32.kicad_pcb (KiCad board)
At the start: 4 copper layers, 34.9 x 48.5 mm, 33 parts, among them J1 USB_C_Receptacle_USB2.0_16P, J2 Conn_01x08, J3 Conn_01x08, U1 USBLC6-2SC6, U2 XC6220B331MR, U3 ESP32-C3-MINI-1

Commit message: Popravljam sedkcije in dodajam slike z handbook
Parts:
- added REF**: Fiducial_1mm_Mask2mm, Fiducial:Fiducial_1mm_Mask2mm, F.Cu at (203.3, 89.3)
Routing:
- net +3.3V: track 15.3 -> 20.8 mm
- net GND: vias 158 -> 157
Changed lines of the file:
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@@
 		)
 	)
+	(footprint "Fiducial:Fiducial_1mm_Mask2mm"
+		(layer "F.Cu")
+		(at 203.3 89.3)
+		(descr "Fiducial, circular marking, 1mm bare copper, 2mm soldermask opening (Level A)")
+		(tags "fiducial")
+		(property "Reference" "REF**"
+			(at 0 -1.95 0)
+			(layer "F.SilkS")
+			(hide yes)
+			(effects
+				(font
+					(size 1 1)
+					(thickness 0.15)
+				)
+			)
+		)
+		(property "Value" "Fiducial_1mm_Mask2mm"
+			(at 0 1.95 0)
+			(layer "F.Fab")
+			(hide yes)
+			(effects
+				(font
+					(size 1 1)
+					(thickness 0.15)
+				)
+			)
+		)
+		(property "Datasheet" ""
+			(at 0 0 0)
+			(layer "F.Fab")
+			(hide yes)
+			(effects
+				(font
+					(size 1.27 1.27)
+				)
+			)
+		)
+		(property "Description" ""
+			(at 0 0 0)
+			(layer "F.Fab")
+			(hide yes)
+			(effects
+				(font
+					(size 1.27 1.27)
+				)
+			)
+		)
+		(property "KiLib_Generator" "fiducial"
+			(at 0 0 0)
+			(layer "F.SilkS")
+			(hide yes)
+			(effects
+				(font
+					(size 1 1)
+					(thickness 0.15)
+				)
+			)
+		)
+		(attr smd exclude_from_bom)
+		(duplicate_pad_numbers_are_jumpers no)
+		(fp_circle
+			(center 0 0)
+			(end 1.25 0)
+			(stroke
+				(width 0.05)
+				(type solid)
+			)
+			(fill no)
+			(layer "F.CrtYd")
+		)
+		(fp_circle
+			(center 0 0)
+			(end 1 0)
+			(stroke
+				(width 0.1)
+				(type solid)
+			)
+			(fill no)
+			(layer "F.Fab")
+		)
+		(fp_text user "${REFERENCE}"
+			(at 0 0 0)
+			(layer "F.Fab")
+			(effects
+				(font
+					(size 0.5 0.5)
+					(thickness 0.08)
+				)
+			)
+		)
+		(pad "" smd circle
+			(at 0 0)
+			(size 1 1)
+			(layers "F.Cu" "F.Mask")
+			(solder_mask_margin 0.5)
+			(clearance 0.6)
+		)
+		(embedded_fonts no)
+	)
 	(footprint "Resistor_SMD:R_0402_1005Metric"
 		(layer "F.Cu")
@@
 	)
 	(via
-		(at 202.6 89.3)
+		(at 226 122.7)
 		(size 0.7)
 		(drill 0.4)
@@
 	)
 	(via
-		(at 226 122.7)
+		(at 226.2 114.6)
 		(size 0.7)
 		(drill 0.4)
@@
 	)
 	(via
-		(at 226.2 114.6)
+		(at 220.5 90.5)
 		(size 0.7)
 		(drill 0.4)
@@
 	)
 	(via
+		(at 218.5 92.4)
+		(size 0.7)
+		(drill 0.4)
+		(layers "F.Cu" "B.Cu")
+		(free yes)
+		(net "GND")
+	)
+	(via
 		(at 216.6 104.1)
 		(size 0.7)
@@
 	)
 	(via
-		(at 204.1 89.3)
-		(size 0.7)
-		(drill 0.4)
-		(layers "F.Cu" "B.Cu")
-		(free yes)
-		(net "GND")
-	)
-	(via
 		(at 208.1 93)
 		(size 0.7)
@@
 	)
 	(via
-		(at 205.9 90)
+		(at 228.2 86.8)
 		(size 0.7)
 		(drill 0.4)
@@
 	)
 	(via
-		(at 228.2 86.8)
+		(at 202.6 87.1)
 		(size 0.7)
 		(drill 0.4)
@@
 	)
 	(via
-		(at 202.6 87.1)
+		(at 228.7 93.8)
 		(size 0.7)
 		(drill 0.4)
@@
 	)
 	(via
-		(at 228.7 93.8)
+		(at 218.4 118)
 		(size 0.7)
 		(drill 0.4)
@@
 	)
 	(via
-		(at 218.4 118)
+		(at 215.1 117.6)
 		(size 0.7)
 		(drill 0.4)
@@
 	)
 	(via
-		(at 215.1 117.6)
+		(at 224.4 113.4)
 		(size 0.7)
 		(drill 0.4)
@@
 	)
 	(via
-		(at 224.4 113.4)
+		(at 218.5 90.5)
 		(size 0.7)
 		(drill 0.4)
@@
 	)
 	(via
-		(at 207 90.9)
-		(size 0.7)
-		(drill 0.4)
-		(layers "F.Cu" "B.Cu")
-		(free yes)
-		(net "GND")
-	)
-	(via
 		(at 230.4 95.3)
 		(size 0.7)
@@
 	)
 	(via
-		(at 205.4 91.2)
-		(size 0.7)
-		(drill 0.4)
-		(layers "F.Cu" "B.Cu")
-		(free yes)
-		(net "GND")
-	)
-	(via
 		(at 202 114.3)
 		(size 0.7)
@@
 	)
 	(via
+		(at 220.5 92.5)
+		(size 0.7)
+		(drill 0.4)
+		(layers "F.Cu" "B.Cu")
+		(free yes)
+		(net "GND")
+	)
+	(via
 		(at 229.6 122.6)
 		(size 0.7)
@@
 	)
 	(segment
+		(start 203 92)
+		(end 204.1 92)
+		(width 0.4)
+		(layer "B.Cu")
+		(net "+3.3V")
+	)
+	(segment
+		(start 204.1 92)
+		(end 207.2 88.9)
+		(width 0.4)
+		(layer "B.Cu")
+		(net "+3.3V")
+	)
+	(segment
 		(start 208 113.1)
 		(end 210.1 113.1)
@@
 		(layer "F.Cu")
 		(hatch edge 0.5)
-		(priority 5)
-		(connect_pads yes
-			(clearance 0.2)
-		)
-		(min_thickness 0.25)
-		(fill yes
-			(thermal_gap 0.5)
-			(thermal_bridge_width 0.5)
-			(island_removal_mode 0)
-		)
-		(polygon
-			(pts
-				(xy 212.4 88) (xy 212.9 88.7) (xy 212.9 90) (xy 211.6 90) (xy 211.6 91.7) (xy 206.2 91.7) (xy 204.3 93.2)
-				(xy 201.7 93.2) (xy 201.7 88)
-			)
-		)
-	)
-	(zone
-		(net "+3.3V")
-		(layer "F.Cu")
-		(hatch edge 0.5)
 		(priority 6)
 		(connect_pads yes
@@
 			)
 		)
+	)
+	(zone
+		(net "+3.3V")
+		(layer "In2.Cu")
+		(hatch edge 0.5)
+		(priority 5)
+		(connect_pads yes
+			(clearance 0.2)
+		)
+		(min_thickness 0.25)
+		(fill yes
+			(thermal_gap 0.5)
+			(thermal_bridge_width 0.5)
+			(island_removal_mode 0)
+		)
+		(polygon
+			(pts
+				(xy 212.4 88) (xy 212.9 88.7) (xy 212.9 90) (xy 211.6 90) (xy 211.6 91.7) (xy 206.2 91.7) (xy 204.3 93.2)
+				(xy 201.7 93.2) (xy 201.7 88)
+			)
+		)
