File: 00-template/FRI-ESP32.kicad_pcb (KiCad board)
At the start: 4 copper layers, 34.9 x 48.5 mm, 0 parts

Commit message: Dodam skripto za export
Parts:
- added BOOT1: SW_Push, fri:SW_SPST_B3U-1000P-B, F.Cu at (228.3, 103.0)
- added C1: 10uF, Capacitor_SMD:C_0805_2012Metric, F.Cu at (223.2, 114.3)
- added C2: 4.7uF, Capacitor_SMD:C_0805_2012Metric, F.Cu at (223.2, 108.1)
- added C3: 100nF, Capacitor_SMD:C_0402_1005Metric, F.Cu at (215.0, 107.0)
- added C4: 100nF, Capacitor_SMD:C_0402_1005Metric, F.Cu at (228.4, 105.2)
- added C5: 100nF, Capacitor_SMD:C_0402_1005Metric, F.Cu at (209.4, 99.7)
- added C6: 100nF, Capacitor_SMD:C_0402_1005Metric, F.Cu at (211.3, 89.0)
- added C7: 10uF, Capacitor_SMD:C_0805_2012Metric, F.Cu at (210.5, 90.5)
- added D1: PESD5V0S1UL, Diode_SMD:D_SOD-882, F.Cu at (215.2, 118.9)
- added D2: LED YELLOW, LED_SMD:LED_0805_2012Metric, F.Cu at (230.4, 91.9)
- added D3: LED GREEN, LED_SMD:LED_0805_2012Metric, F.Cu at (230.4, 87.8)
- added J1: USB_C_Receptacle_USB2.0_16P, fri:USB_C_Receptacle_G-Switch_GT-USB-7010ASV, F.Cu at (218.0, 124.4)
- added J2: Conn_01x08, Connector_PinHeader_2.54mm:PinHeader_1x08_P2.54mm_Vertical, F.Cu at (233.1, 103.2)
- added J3: Conn_01x08, Connector_PinHeader_2.54mm:PinHeader_1x08_P2.54mm_Vertical, F.Cu at (203.3, 103.2)
- added R1: 5.1K, Resistor_SMD:R_0402_1005Metric, F.Cu at (222.0, 118.2)
- added R10: 10K, Resistor_SMD:R_0402_1005Metric, F.Cu at (222.5, 98.1)
- added R2: 5.1K, Resistor_SMD:R_0402_1005Metric, F.Cu at (215.3, 117.2)
- added R3: 10K, Resistor_SMD:R_0402_1005Metric, F.Cu at (222.5, 116.0)
- added R4: 10K, Resistor_SMD:R_0402_1005Metric, F.Cu at (216.3, 102.5)
- added R5: 10K, Resistor_SMD:R_0402_1005Metric, F.Cu at (228.6, 100.7)
- added R6: 330, Resistor_SMD:R_0402_1005Metric, F.Cu at (230.7, 93.5)
- added R7: 330, Resistor_SMD:R_0402_1005Metric, F.Cu at (230.8, 89.4)
- added R8: 10K, Resistor_SMD:R_0402_1005Metric, F.Cu at (209.4, 98.7)
- added R9: 10K, Resistor_SMD:R_0402_1005Metric, F.Cu at (210.9, 92.3)
- added REF**: Fiducial_1mm_Mask2mm, fri:Fiducial_1mm_Mask2mm, F.Cu at (232.8, 126.1)
- added REF**: Fiducial_1mm_Mask2mm, fri:Fiducial_1mm_Mask2mm, F.Cu at (203.4, 125.9)
- added REF**: Fiducial_1mm_Mask2mm, fri:Fiducial_1mm_Mask2mm, F.Cu at (203.1, 87.7)
- added RESET1: SW_Push, fri:SW_SPST_B3U-1000P-B, F.Cu at (207.0, 96.4)
- added U1: XC6220B331MR, fri:SOT-23-5, F.Cu at (223.0, 111.2)
- added U2: USBLC6-2SC6, fri:SOT-23-6, F.Cu at (218.6, 117.5)
- added U3: ESP32-C3-MINI-1, fri:ESP32-C3-MINI-1, F.Cu at (219.1, 88.6)
- added USRBUTTON1: SW_Push, fri:SW_SPST_B3U-1000P-B, F.Cu at (214.9, 104.8)
Routing:
- net GND: track 0.00 -> 95.6 mm, vias 0 -> 49
- net GPIO3: track 0.00 -> 34.0 mm, vias 0 -> 2
- net GPIO0: track 0.00 -> 32.9 mm, vias 0 -> 2
- net GPIO1: track 0.00 -> 31.2 mm, vias 0 -> 2
- net USBD+: track 0.00 -> 29.0 mm
- net USBD-: track 0.00 -> 28.2 mm
- net TXD: track 0.00 -> 27.1 mm
- net VBUS: track 0.00 -> 25.5 mm, vias 0 -> 6
- net +3.3V: track 0.00 -> 23.3 mm, vias 0 -> 12
- net GPIO4: track 0.00 -> 23.3 mm, vias 0 -> 2
- net RXD: track 0.00 -> 21.8 mm, vias 0 -> 2
- net GPIO5: track 0.00 -> 21.2 mm, vias 0 -> 2
- net GPIO9_BOOT: track 0.00 -> 15.5 mm, vias 0 -> 2
- net LED1: track 0.00 -> 13.2 mm, vias 0 -> 2
- net USER_BTN: track 0.00 -> 11.6 mm
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- added copper zone on In2.Cu, net +3.3V
- added copper zone on B.Cu, net GND
- added copper zone on F.Cu, net GND
- added copper zone on In2.Cu, net VBUS
