File: 00-template/digital.kicad_sch (KiCad schematic)
At the start: 0 parts

Commit message: Dodam skripto za export
Parts:
- added BOOT1, RESET1, USRBUTTON1: SW_Push, fri:SW_SPST_B3U-1000P-B, symbol fri:SW_Push
- added C3, C4, C5, C6: 100nF, Capacitor_SMD:C_0402_1005Metric, symbol Device:C
- added C7: 10uF, Capacitor_SMD:C_0805_2012Metric, symbol Device:C
- added D2: LED YELLOW, LED_SMD:LED_0805_2012Metric, symbol fri:LED
- added D3: LED GREEN, LED_SMD:LED_0805_2012Metric, symbol fri:LED
- added J2, J3: Conn_01x08, Connector_PinHeader_2.54mm:PinHeader_1x08_P2.54mm_Vertical, symbol fri:Conn_01x08
- added R10, R4, R5, R8, R9: 10K, Resistor_SMD:R_0402_1005Metric, symbol Device:R
- added R6, R7: 330, Resistor_SMD:R_0402_1005Metric, symbol Device:R
- added U3: ESP32-C3-MINI-1, fri:ESP32-C3-MINI-1, symbol fri:ESP32-C3-MINI-1
Connections:
- new net: D3.2 (A), R7.2
- new net: D2.2 (A), R6.2
- new net +3.3V: C6.1, C7.1, J3.1 (Pin_1), J3.2 (Pin_2), J3.3 (Pin_3), R10.1, R4.1, R5.1, R6.1, R7.1, R8.1, R9.1, U3.3 (3V3)
- new net EN: C5.1, R8.2, RESET1.2, U3.8 (EN/CHIP_PU)
- new net GND: BOOT1.1, C3.2, C4.2, C5.2, C6.2, C7.2, J2.3 (Pin_3), J3.5 (Pin_5), J3.6 (Pin_6), J3.7 (Pin_7), J3.8 (Pin_8), RESET1.1, U3.1 (GND), U3.11 (GND), U3.14 (GND), U3.2 (GND), U3.36 (GND), U3.37 (GND), U3.38 (GND), U3.39 (GND), U3.40 (GND), U3.41 (GND), U3.42 (GND), U3.43 (GND), U3.44 (GND), U3.45 (GND), U3.46 (GND), U3.47 (GND), U3.48 (GND), U3.49 (GND), U3.50 (GND), U3.51 (GND), U3.52 (GND), U3.53 (GND), USRBUTTON1.1
- new net GPIO0: J2.8 (Pin_8), U3.12 (GPIO0/ADC1_CH0/XTAL_32K_P)
- new net GPIO1: J2.7 (Pin_7), U3.13 (GPIO1/ADC1_CH1/XTAL_32K_N)
- new net GPIO2_BOOT: R9.2, U3.5 (GPIO2/ADC1_CH2)
- new net GPIO3: J2.6 (Pin_6), U3.6 (GPIO3/ADC1_CH3)
- new net GPIO4: J2.5 (Pin_5), U3.18 (GPIO4/ADC1_CH4)
- new net GPIO5: J2.4 (Pin_4), U3.19 (GPIO5/ADC2_CH0)
- new net GPIO8_BOOT: R10.2, U3.22 (GPIO8)
- new net GPIO9_BOOT: BOOT1.2, C4.1, R5.2, U3.23 (GPIO9)
- new net LED0: D2.1 (K), U3.20 (GPIO6)
- new net LED1: D3.1 (K), U3.21 (GPIO7)
- new net RXD: J2.2 (Pin_2), U3.30 (GPIO20/U0RXD)
- new net TXD: J2.1 (Pin_1), U3.31 (GPIO21/U0TXD)
- new net USBD+: U3.27 (GPIO19/USB_D+)
- new net USBD-: U3.26 (GPIO18/USB_D-)
- new net USER_BTN: C3.1, R4.2, U3.16 (GPIO10), USRBUTTON1.2
- new net VBUS: J3.4 (Pin_4)
