File: 00-template/power.kicad_sch (KiCad schematic)
At the start: 0 parts

Commit message: Dodam skripto za export
Parts:
- added C1: 10uF, Capacitor_SMD:C_0805_2012Metric, symbol Device:C
- added C2: 4.7uF, Capacitor_SMD:C_0805_2012Metric, symbol Device:C
- added D1: PESD5V0S1UL, Diode_SMD:D_SOD-882, symbol fri:PESD5V0S1UL
- added J1: USB_C_Receptacle_USB2.0_16P, fri:USB_C_Receptacle_G-Switch_GT-USB-7010ASV, symbol fri:USB_C_Receptacle_USB2.0_16P
- added R1, R2: 5.1K, Resistor_SMD:R_0402_1005Metric, symbol Device:R
- added R3: 10K, Resistor_SMD:R_0402_1005Metric, symbol Device:R
- added U1: XC6220B331MR, fri:SOT-23-5, symbol fri:XC6220B331MR
- added U2: USBLC6-2SC6, fri:SOT-23-6, symbol fri:USBLC6-2SC6
Connections:
- new net: R3.2, U1.3 (CE)
- new net: J1.A5 (CC1), R2.1
- new net: J1.A6 (D+), J1.B6 (D+), U2.3 (I/O2)
- new net: J1.A7 (D-), J1.B7 (D-), U2.1 (I/O1)
- new net: J1.B5 (CC2), R1.1
- new net +3.3V: C2.1, U1.5 (VOUT)
- new net GND: C1.2, C2.2, D1.2 (A), J1.A1 (GND), J1.A12 (GND), J1.B1 (GND), J1.B12 (GND), J1.SH (SHIELD), R1.2, R2.2, U1.2 (GND), U2.2 (GND)
- new net USBD+: U2.4 (I/O2)
- new net USBD-: U2.6 (I/O1)
- new net VBUS: C1.1, D1.1 (K), J1.A4 (VBUS), J1.A9 (VBUS), J1.B4 (VBUS), J1.B9 (VBUS), R3.1, U1.1 (VIN), U2.5 (VBUS)
- no-connect marks 0 -> 2
Other:
- note added: "LDO 3.3V"
- note added: "USB-C Power delivery"
